Commit message: remove build files
remove build files

File: src/my_robot/urdf/my_robot_2WL_Color.xacro (robot description, xacro)
@@ -69,5 +69,5 @@
   </link>
   <joint name="left_wheel_hinge" type="continuous">
-    <origin xyz="0.15 0.25 0" rpy="0 0 0" />
+    <origin xyz="0 0.15 0" rpy="0 0 0" />
     <parent link="chassis"/>
     <child link="left_wheel" />
@@ -77,23 +77,7 @@
   </joint>
   <joint name="right_wheel_hinge" type="continuous">
-    <origin xyz="0.15 -0.25 0" rpy="0 0 0" />
+    <origin xyz="0 -0.15 0" rpy="0 0 0" />
     <parent link="chassis"/>
     <child link="right_wheel" />
-    <axis xyz="0 1 0" rpy="0 0 0"/>
-    <limit effort="10000" velocity="1000"/>
-    <dynamics damping="1.0" friction="1.0"/>
-  </joint>
-  <joint name="left_back_wheel_hinge" type="continuous">
-    <origin xyz="-0.15 0.25 0" rpy="0 0 0" />
-    <parent link="chassis"/>
-    <child link="left_back_wheel" />
-    <axis xyz="0 1 0" rpy="0 0 0"/>
-    <limit effort="10000" velocity="1000"/>
-    <dynamics damping="1.0" friction="1.0"/>
-  </joint>
-  <joint name="right_back_wheel_hinge" type="continuous">
-    <origin xyz="-0.15 -0.25 0" rpy="0 0 0" />
-    <parent link="chassis"/>
-    <child link="right_back_wheel" />
     <axis xyz="0 1 0" rpy="0 0 0"/>
     <limit effort="10000" velocity="1000"/>
@@ -146,50 +130,4 @@
     </visual>
   </link>
-  <link name='right_back_wheel'>
-    <pos>0 0 0 0 0 0</pos>
-    <inertial>
-      <mass value="5.0"/>
-      <inertia
-          ixx="0.1" ixy="0" ixz="0"
-          iyy="0.1" iyz="0"
-          izz="0.1"
-      />
-    </inertial>
-    <collision name='collision'>
-      <origin xyz="0 0 0" rpy=" 0 1.5707 1.5707"/>
-      <geometry>
-        <cylinder radius="0.1" length="0.05"/>
-      </geometry>
-    </collision>
-    <visual name='right_back_wheel_visual'>
-      <origin xyz="0 0 0" rpy=" 0 1.5707 1.5707"/>
-      <geometry>
-        <cylinder radius="0.1" length="0.05"/>
-      </geometry>
-    </visual>
-  </link>
-  <link name='left_back_wheel'>
-    <pos>0 0 0 0 0 0</pos>
-    <inertial>
-      <mass value="5.0"/>
-      <inertia
-          ixx="0.1" ixy="0" ixz="0"
-          iyy="0.1" iyz="0"
-          izz="0.1"
-      />
-    </inertial>
-    <collision name='collision'>
-      <origin xyz="0 0 0" rpy=" 0 1.5707 1.5707"/>
-      <geometry>
-        <cylinder radius="0.1" length="0.05"/>
-      </geometry>
-    </collision>
-    <visual name='left_back_wheel_visual'>
-      <origin xyz="0 0 0" rpy=" 0 1.5707 1.5707"/>
-      <geometry>
-        <cylinder radius="0.1" length="0.05"/>
-      </geometry>
-    </visual>
-  </link>
   <link name='chassis'>
     <pose>0 0 0.1 0 0 0</pose>
@@ -206,5 +144,5 @@
       <origin xyz="0 0 0" rpy=" 0 0 0"/>
       <geometry>
-        <box size=".4 .4 .1"/>
+        <box size=".4 .2 .1"/>
       </geometry>
     </collision>
@@ -212,5 +150,5 @@
       <origin xyz="0 0 0" rpy=" 0 0 0"/>
       <geometry>
-        <box size=".4 .4 .1"/>
+        <box size=".4 .2 .1"/>
       </geometry>
     </visual>

File: src/my_robot/urdf/my_robot_4W.xacro (robot description, xacro)
@@ -69,5 +69,5 @@
   </link>
   <joint name="left_wheel_hinge" type="continuous">
-    <origin xyz="0.15 0.25 0" rpy="0 0 0" />
+    <origin xyz="0.15 0.15 0" rpy="0 0 0" />
     <parent link="chassis"/>
     <child link="left_wheel" />
@@ -77,5 +77,5 @@
   </joint>
   <joint name="right_wheel_hinge" type="continuous">
-    <origin xyz="0.15 -0.25 0" rpy="0 0 0" />
+    <origin xyz="0.15 -0.15 0" rpy="0 0 0" />
     <parent link="chassis"/>
     <child link="right_wheel" />
@@ -85,5 +85,5 @@
   </joint>
   <joint name="left_back_wheel_hinge" type="continuous">
-    <origin xyz="-0.15 0.25 0" rpy="0 0 0" />
+    <origin xyz="-0.15 0.15 0" rpy="0 0 0" />
     <parent link="chassis"/>
     <child link="left_back_wheel" />
@@ -93,5 +93,5 @@
   </joint>
   <joint name="right_back_wheel_hinge" type="continuous">
-    <origin xyz="-0.15 -0.25 0" rpy="0 0 0" />
+    <origin xyz="-0.15 -0.15 0" rpy="0 0 0" />
     <parent link="chassis"/>
     <child link="right_back_wheel" />
@@ -206,5 +206,5 @@
       <origin xyz="0 0 0" rpy=" 0 0 0"/>
       <geometry>
-        <box size=".4 .4 .1"/>
+        <box size=".4 .2 .1"/>
       </geometry>
     </collision>
@@ -212,5 +212,5 @@
       <origin xyz="0 0 0" rpy=" 0 0 0"/>
       <geometry>
-        <box size=".4 .4 .1"/>
+        <box size=".4 .2 .1"/>
       </geometry>
     </visual>
