Commit message: update drive service response
response to include the linear and angular information

File: src/my_robot/urdf/my_robot.xacro (robot description, xacro)
@@ -69,5 +69,5 @@
   </link>
   <joint name="left_wheel_hinge" type="continuous">
-    <origin xyz="0.15 0.25 0" rpy="0 0 0" />
+    <origin xyz="0.15 0.15 0" rpy="0 0 0" />
     <parent link="chassis"/>
     <child link="left_wheel" />
@@ -77,5 +77,5 @@
   </joint>
   <joint name="right_wheel_hinge" type="continuous">
-    <origin xyz="0.15 -0.25 0" rpy="0 0 0" />
+    <origin xyz="0.15 -0.15 0" rpy="0 0 0" />
     <parent link="chassis"/>
     <child link="right_wheel" />
@@ -85,5 +85,5 @@
   </joint>
   <joint name="left_back_wheel_hinge" type="continuous">
-    <origin xyz="-0.15 0.25 0" rpy="0 0 0" />
+    <origin xyz="-0.15 0.15 0" rpy="0 0 0" />
     <parent link="chassis"/>
     <child link="left_back_wheel" />
@@ -93,5 +93,5 @@
   </joint>
   <joint name="right_back_wheel_hinge" type="continuous">
-    <origin xyz="-0.15 -0.25 0" rpy="0 0 0" />
+    <origin xyz="-0.15 -0.15 0" rpy="0 0 0" />
     <parent link="chassis"/>
     <child link="right_back_wheel" />
@@ -116,5 +116,5 @@
       </geometry>
     </collision>
-    <visual name='right_wheel_visual'>
+    <visual name='visual'>
       <origin xyz="0 0 0" rpy=" 0 1.5707 1.5707"/>
       <geometry>
@@ -139,5 +139,5 @@
       </geometry>
     </collision>
-    <visual name='left_wheel_visual'>
+    <visual name='visual'>
       <origin xyz="0 0 0" rpy=" 0 1.5707 1.5707"/>
       <geometry>
@@ -162,5 +162,5 @@
       </geometry>
     </collision>
-    <visual name='right_back_wheel_visual'>
+    <visual name='visual'>
       <origin xyz="0 0 0" rpy=" 0 1.5707 1.5707"/>
       <geometry>
@@ -185,5 +185,5 @@
       </geometry>
     </collision>
-    <visual name='left_back_wheel_visual'>
+    <visual name='visual'>
       <origin xyz="0 0 0" rpy=" 0 1.5707 1.5707"/>
       <geometry>
@@ -206,5 +206,5 @@
       <origin xyz="0 0 0" rpy=" 0 0 0"/>
       <geometry>
-        <box size=".4 .4 .1"/>
+        <box size=".4 .2 .1"/>
       </geometry>
     </collision>
@@ -212,5 +212,5 @@
       <origin xyz="0 0 0" rpy=" 0 0 0"/>
       <geometry>
-        <box size=".4 .4 .1"/>
+        <box size=".4 .2 .1"/>
       </geometry>
     </visual>

Commit message: update robot
include color, chassis dimension changed to square (better in turn) and have 4 wheel with skid control

File: src/my_robot/urdf/my_robot.xacro (robot description, xacro)
@@ -69,5 +69,5 @@
   </link>
   <joint name="left_wheel_hinge" type="continuous">
-    <origin xyz="0.15 0.15 0" rpy="0 0 0" />
+    <origin xyz="0.15 0.25 0" rpy="0 0 0" />
     <parent link="chassis"/>
     <child link="left_wheel" />
@@ -77,5 +77,5 @@
   </joint>
   <joint name="right_wheel_hinge" type="continuous">
-    <origin xyz="0.15 -0.15 0" rpy="0 0 0" />
+    <origin xyz="0.15 -0.25 0" rpy="0 0 0" />
     <parent link="chassis"/>
     <child link="right_wheel" />
@@ -85,5 +85,5 @@
   </joint>
   <joint name="left_back_wheel_hinge" type="continuous">
-    <origin xyz="-0.15 0.15 0" rpy="0 0 0" />
+    <origin xyz="-0.15 0.25 0" rpy="0 0 0" />
     <parent link="chassis"/>
     <child link="left_back_wheel" />
@@ -93,5 +93,5 @@
   </joint>
   <joint name="right_back_wheel_hinge" type="continuous">
-    <origin xyz="-0.15 -0.15 0" rpy="0 0 0" />
+    <origin xyz="-0.15 -0.25 0" rpy="0 0 0" />
     <parent link="chassis"/>
     <child link="right_back_wheel" />
@@ -116,5 +116,5 @@
       </geometry>
     </collision>
-    <visual name='visual'>
+    <visual name='right_wheel_visual'>
       <origin xyz="0 0 0" rpy=" 0 1.5707 1.5707"/>
       <geometry>
@@ -139,5 +139,5 @@
       </geometry>
     </collision>
-    <visual name='visual'>
+    <visual name='left_wheel_visual'>
       <origin xyz="0 0 0" rpy=" 0 1.5707 1.5707"/>
       <geometry>
@@ -162,5 +162,5 @@
       </geometry>
     </collision>
-    <visual name='visual'>
+    <visual name='right_back_wheel_visual'>
       <origin xyz="0 0 0" rpy=" 0 1.5707 1.5707"/>
       <geometry>
@@ -185,5 +185,5 @@
       </geometry>
     </collision>
-    <visual name='visual'>
+    <visual name='left_back_wheel_visual'>
       <origin xyz="0 0 0" rpy=" 0 1.5707 1.5707"/>
       <geometry>
@@ -206,5 +206,5 @@
       <origin xyz="0 0 0" rpy=" 0 0 0"/>
       <geometry>
-        <box size=".4 .2 .1"/>
+        <box size=".4 .4 .1"/>
       </geometry>
     </collision>
@@ -212,5 +212,5 @@
       <origin xyz="0 0 0" rpy=" 0 0 0"/>
       <geometry>
-        <box size=".4 .2 .1"/>
+        <box size=".4 .4 .1"/>
       </geometry>
     </visual>
